Commit message: Added control script

File: urdf/materials.xacro (robot description, xacro)
@@ -7,3 +7,12 @@
   <color rgba="0.6274509803921569 0.6274509803921569 0.6274509803921569 1.0"/>
 </material>
+<material name="base_colour">
+  <color rgba="1.0 0.4 0.0 1.0"/>
+</material>
+<material name="arm1_colour">
+  <color rgba="0.0 1.0 1.0 1.0"/>
+</material>
+<material name="arm2_colour">
+  <color rgba="1.0 0.0 1.0 1.0"/>
+</material>
 </robot>

File: urdf/rr_bot.xacro (robot description, xacro)
@@ -15,5 +15,5 @@
       <mesh filename="package://rr_bot_description/meshes/base_link.stl" scale="0.001 0.001 0.001"/>
     </geometry>
-    <material name="steel_satin"/>
+    <material name="base_colour"/>
   </visual>
   <collision>
@@ -35,5 +35,5 @@
       <mesh filename="package://rr_bot_description/meshes/arm1_v5_1.stl" scale="0.001 0.001 0.001"/>
     </geometry>
-    <material name="steel_satin"/>
+    <material name="arm1_colour"/>
   </visual>
   <collision>
@@ -55,5 +55,5 @@
       <mesh filename="package://rr_bot_description/meshes/arm2_v4_1.stl" scale="0.001 0.001 0.001"/>
     </geometry>
-    <material name="steel_satin"/>
+    <material name="arm2_colour"/>
   </visual>
   <collision>
